Commit message: Updated files in elite_description folder

File: elite_description/urdf/_d435.urdf.xacro (robot description, xacro)
@@ -66,5 +66,6 @@
         <origin xyz="0 ${-d435_cam_depth_py} 0" rpy="0 0 0"/>
         <geometry>
-          <box size="${d435_cam_depth} ${d435_cam_width} ${d435_cam_height}"/>
+          <!-- <box size="${d435_cam_depth} ${d435_cam_width} ${d435_cam_height}"/> -->
+          <box size="0.001 0.001 0.001"/>
         </geometry>
       </collision>

File: elite_description/urdf/ec63_description.urdf (robot description, URDF)
Before this commit: robot ec63, 9 links, 8 joints
Links:
- added link camera_lin, mass 0.001
- added link camera_mount, mass 0.010466; collision mesh filename=package://elite_description/meshes/ec66/Intel_D435_clamp(1)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 scale=0.001 0.001 0.001; visual mesh filename=package://elite_description/meshes/ec66/Intel_D435_clamp(1)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 scale=0.001 0.001 0.001
Joints:
- added joint camera_lin: type fixed, parent camera_mount, child camera_lin, origin xyz=0.065 0.035 0.00 rpy=-1.57 3.14 0, axis 0 0 0
- added joint camera_mount_joint: type fixed, parent flan, child camera_mount, origin xyz=0 0 0 rpy=1.57 0 0, axis 0 0 0

File: elite_description/urdf/ec66_description.xacro (robot description, xacro)
@@ -236,5 +236,5 @@
     <inertial>
       <origin xyz="-0.0051042 0.00088494 -0.00052221" rpy="0 0 0" />
-      <mass value="0.10466" />
+      <mass value="0.010466" />
       <inertia ixx="0.00061835" ixy="0.00024116" ixz="-6.2654E-05" iyy="1.00441" iyz="1.3293E-05" izz="1.000143" />
     </inertial>
@@ -264,22 +264,7 @@
     <inertial>
       <origin xyz="-0.0051042 0.00088494 -0.00052221" rpy="0 0 0" />
-      <mass value="0.10466" />
-      <inertia ixx="0.00061835" ixy="0.00024116" ixz="-6.2654E-05" iyy="1.00441" iyz="1.3293E-05" izz="1.000143" />
-    </inertial>
-    <visual>
-      <origin xyz="0 0 0" rpy="0 0 0" />
-      <geometry>
-        <box size="0 0 0" />
-      </geometry>
-      <material name="">
-        <color rgba="1 1 1 1" />
-      </material>
-    </visual>
-    <collision>
-      <origin xyz="0 0 0" rpy="0 0 0" />
-      <geometry>
-        <box size="0 0 0" />
-      </geometry>
-    </collision>
+      <mass value="0.001" />
+      <inertia ixx="0.0000061835" ixy="0.0000024116" ixz="-6.2654E-07" iyy="1.00441" iyz="1.3293E-05" izz="1.000143" />
+    </inertial>
     </link>
     <joint name="camera_lin" type="fixed">
